Commit message: fix: Fix orientation of base link to make it consistent with Frontier v7 URDF following ROS REP 103

File: urdf/magnet.urdf.xacro (robot description, xacro)
@@ -13,5 +13,5 @@
             <color rgba="0.3 0.3 0.3 1"/>
         </material>
-        <origin xyz="-0.055 0.055 0" rpy="${pi/2} 0 0"/>
+        <origin xyz="-0.055 -0.055 0" rpy="${pi/2} 0 ${pi/2}"/>
         <geometry>
           <mesh filename="file://$(find magnet_description)/meshes/visual/case.stl" scale="0.001 0.001 0.001"/>
@@ -21,5 +21,5 @@
     <xacro:include filename="$(find microstrain_inertial_description)/urdf/gx5_15.urdf.xacro"/>
     <xacro:gx5_15 name="${prefix}gx5_15" parent="${prefix}magnet">
-      <origin xyz="0.0 -0.0058 0.0574" rpy="0 0 ${-pi/2}" />
+      <origin xyz="0.0058 0.0 0.0574" rpy="0 0 0" />
     </xacro:gx5_15>
     <link name="heatsink">
@@ -28,5 +28,5 @@
             <color rgba="0.7 0.7 0.7 1"/>
         </material>
-        <origin xyz="-0.055 0.055 0" rpy="${pi/2} 0 0"/>
+        <origin xyz="-0.055 -0.055 0" rpy="${pi/2} 0 ${pi/2}"/>
         <geometry>
           <mesh filename="file://$(find magnet_description)/meshes/visual/heatsink.stl" scale="0.001 0.001 0.001"/>
@@ -41,5 +41,5 @@
     <xacro:include filename="$(find hesai_description)/urdf/hesai_qt64.urdf.xacro"/>
     <xacro:hesai_qt64 name="${prefix}hesai_qt64" parent="${prefix}magnet" simulation="${simulation}" use_gpu="${use_gpu}">
-      <origin xyz="0 0 0.072" rpy="0 0 0" />
+      <origin xyz="0 0 0.072" rpy="0 0 ${pi/2}" />
     </xacro:hesai_qt64>
   </xacro:macro>

Commit message: fix: Change link naming convention to be identical to Frontier v7 and add dummy link for Magnet base

File: urdf/magnet.urdf.xacro (robot description, xacro)
@@ -3,10 +3,10 @@
   <xacro:macro name="magnet" params="parent *origin prefix:='' name:=magnet
                                      simulation:=false use_gpu:=true">
-    <joint name="${parent}_to_${prefix}magnet" type="fixed">
+    <joint name="${parent}_to_${prefix}magnet_mount" type="fixed">
       <xacro:insert_block name="origin"/>
       <parent link="${parent}" />
-      <child link="${prefix}magnet" />
+      <child link="${prefix}magnet_mount" />
     </joint>
-    <link name="${prefix}magnet">
+    <link name="${prefix}magnet_mount">
       <visual>
         <material name="darkgrey">
@@ -20,5 +20,5 @@
     </link>
     <xacro:include filename="$(find microstrain_inertial_description)/urdf/gx5_15.urdf.xacro"/>
-    <xacro:gx5_15 name="${prefix}gx5_15" parent="${prefix}magnet">
+    <xacro:gx5_15 name="${prefix}gx5_15" parent="${prefix}magnet_mount">
       <origin xyz="0.0058 0.0 0.0574" rpy="0 0 0" />
     </xacro:gx5_15>
@@ -34,13 +34,21 @@
       </visual>
     </link>
-    <joint name="${prefix}magnet_to_${prefix}heatsink" type="fixed">
+    <joint name="${prefix}magnet_mount_to_${prefix}heatsink" type="fixed">
       <origin xyz="0 0 0.069" rpy="0 0 0" />
-      <parent link="${prefix}magnet" />
+      <parent link="${prefix}magnet_mount" />
       <child link="${prefix}heatsink" />
     </joint>
     <xacro:include filename="$(find hesai_description)/urdf/hesai_qt64.urdf.xacro"/>
-    <xacro:hesai_qt64 name="${prefix}hesai_qt64" parent="${prefix}magnet" simulation="${simulation}" use_gpu="${use_gpu}">
-      <origin xyz="0 0 0.072" rpy="0 0 ${pi/2}" />
+    <!-- The height of the Magnet 3D-printed case: From bottom of case to the top of the lidar plate -->
+    <xacro:property name="magnet_case_height" value="0.072"/>
+    <xacro:hesai_qt64 name="${prefix}hesai_qt64" parent="${prefix}magnet_mount" simulation="${simulation}" use_gpu="${use_gpu}">
+      <origin xyz="0 0 ${magnet_case_height}" rpy="0 0 ${pi/2}" />
     </xacro:hesai_qt64>
+    <link name="${prefix}magnet_base" />
+    <joint name="${prefix}magnet_mount_to_${prefix}magnet_base" type="fixed">
+      <parent link="${prefix}magnet_mount" />
+      <child link="${prefix}magnet_base" />
+      <origin xyz="0 0 ${magnet_case_height}" rpy="0 0 0" />
+    </joint>
   </xacro:macro>
 </robot>

File: urdf/standalone.urdf.xacro (robot description, xacro)
@@ -5,6 +5,6 @@
   <xacro:arg name="use_gpu" default="true" />
   <xacro:include filename="$(find magnet_description)/urdf/magnet.urdf.xacro" />
-  <link name="base"/>
-  <xacro:magnet parent="base" prefix="$(arg prefix)" simulation="$(arg simulation)" use_gpu="$(arg use_gpu)" >
+  <link name="root"/>
+  <xacro:magnet parent="root" prefix="$(arg prefix)" simulation="$(arg simulation)" use_gpu="$(arg use_gpu)" >
     <origin xyz="0 0 0" rpy="0 0 0" />
   </xacro:magnet>

Commit message: use package:// rather than file:// so models load over network

File: urdf/magnet.urdf.xacro (robot description, xacro)
@@ -15,5 +15,5 @@
         <origin xyz="-0.055 -0.055 0" rpy="${pi/2} 0 ${pi/2}"/>
         <geometry>
-          <mesh filename="file://$(find magnet_description)/meshes/visual/case.stl" scale="0.001 0.001 0.001"/>
+          <mesh filename="package://magnet_description/meshes/visual/case.stl" scale="0.001 0.001 0.001"/>
         </geometry>
       </visual>
@@ -30,5 +30,5 @@
         <origin xyz="-0.055 -0.055 0" rpy="${pi/2} 0 ${pi/2}"/>
         <geometry>
-          <mesh filename="file://$(find magnet_description)/meshes/visual/heatsink.stl" scale="0.001 0.001 0.001"/>
+          <mesh filename="package://magnet_description/meshes/visual/heatsink.stl" scale="0.001 0.001 0.001"/>
         </geometry>
       </visual>
